File: pcb/pcb.kicad_pcb (KiCad board)
At the start: 2 copper layers, 40 x 47 mm, 8 parts, among them SW1 SW_SPDT, U1 Pimoroni_LiPo_Amigo, U2 Timecube_Accelerometer, U3 Tiny2040, U5 E-ink_Driver

Commit message: pcb updates for 1.0
Parts:
- moved U2 9.96 mm to (110.7, 108.0), turned to 180 degrees
- moved U3 2.62 mm to (130.8, 82.0)
Connections:
- U2 pad 2: Net-(U2-Pad2) -> Net-(U3-Pad7)
- U2 pad 4: Net-(U2-Pad4) -> Net-(U3-Pad5)
- U3 pad 5: Net-(U2-Pad2) -> Net-(U3-Pad5)
- U3 pad 7: Net-(U2-Pad4) -> Net-(U3-Pad7)
Routing:
- net Net-(U2-Pad4): track 31.0 -> 0.00 mm
- net Net-(U2-Pad2): track 31.0 -> 0.00 mm
- net Net-(U3-Pad5): track 0.00 -> 27.0 mm
- net Net-(U3-Pad7): track 0.00 -> 26.2 mm
- net /VCC: track 32.6 -> 37.6 mm
- net Net-(U2-Pad3): track 31.0 -> 26.6 mm
- net Net-(U3-Pad11): track 16.4 -> 13.7 mm
- net Net-(U3-Pad16): track 32.7 -> 30.1 mm
- net Net-(U3-Pad15): track 29.1 -> 26.5 mm
- net Net-(U3-Pad14): track 25.5 -> 22.9 mm
- net Net-(U3-Pad13): track 21.9 -> 19.3 mm
- net Net-(U3-Pad12): track 18.3 -> 15.7 mm
- net Net-(U1-Pad2): track 45.9 -> 44.3 mm
- net Net-(R1-Pad2): track 41.2 -> 40.2 mm
- net Net-(D1-Pad1): track 36.2 -> 35.1 mm
Other:
- board text added: "ON"
- board text added: "v1.0"
- board text removed: "v0.3"
