File: pcb/pcb.kicad_sch (KiCad schematic)
At the start: 8 parts, among them SW1 SW_SPDT, U1 Pimoroni_LiPo_Amigo, U2 Timecube_Accelerometer, U3 Tiny2040, U5 E-ink_Driver

Commit message: pcb updates for 1.0
Connections:
- net at U2.2 (X): now also U3.7 (GP26); no longer U3.5 (GP28)
- net at U2.4 (Z): now also U3.5 (GP28); no longer U3.7 (GP26)
Changed lines of the file:
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@@
-    (stroke (width 0) (type default) (color 0 0 0 0))
-  )
-  (wire (pts (xy 133.35 95.25) (xy 144.78 95.25))
     (stroke (width 0) (type default) (color 0 0 0 0))
   )
@@
     (stroke (width 0) (type default) (color 0 0 0 0))
   )
+  (wire (pts (xy 133.35 95.25) (xy 138.43 95.25))
+    (stroke (width 0) (type default) (color 0 0 0 0))
+  )
   (wire (pts (xy 119.38 58.42) (xy 182.88 58.42))
     (stroke (width 0) (type default) (color 0 0 0 0))
@@
   )
   (wire (pts (xy 177.8 95.25) (xy 189.23 95.25))
+    (stroke (width 0) (type default) (color 0 0 0 0))
+  )
+  (wire (pts (xy 138.43 102.87) (xy 144.78 102.87))
     (stroke (width 0) (type default) (color 0 0 0 0))
   )
@@
     (stroke (width 0) (type default) (color 0 0 0 0))
   )
+  (wire (pts (xy 138.43 95.25) (xy 138.43 102.87))
+    (stroke (width 0) (type default) (color 0 0 0 0))
+  )
   (wire (pts (xy 182.88 58.42) (xy 182.88 106.68))
+    (stroke (width 0) (type default) (color 0 0 0 0))
+  )
+  (wire (pts (xy 133.35 102.87) (xy 135.89 102.87))
+    (stroke (width 0) (type default) (color 0 0 0 0))
+  )
+  (wire (pts (xy 135.89 93.98) (xy 144.78 93.98))
     (stroke (width 0) (type default) (color 0 0 0 0))
   )
@@
   )
   (wire (pts (xy 177.8 87.63) (xy 189.23 87.63))
-    (stroke (width 0) (type default) (color 0 0 0 0))
-  )
-  (wire (pts (xy 133.35 102.87) (xy 144.78 102.87))
     (stroke (width 0) (type default) (color 0 0 0 0))
   )
@@
     (stroke (width 0) (type default) (color 0 0 0 0))
   )
+  (wire (pts (xy 135.89 102.87) (xy 135.89 93.98))
+    (stroke (width 0) (type default) (color 0 0 0 0))
+  )
   (wire (pts (xy 127 60.96) (xy 127 64.77))
     (stroke (width 0) (type default) (color 0 0 0 0))
@@
     (stroke (width 0) (type default) (color 0 0 0 0))
   )
+  (wire (pts (xy 144.78 93.98) (xy 144.78 95.25))
+    (stroke (width 0) (type default) (color 0 0 0 0))
+  )
